File: pcb_picokeyboard.kicad_sch (KiCad schematic)
At the start: 9 parts, among them J1 PICO, J2 502790-3091

Commit message: 2
Connections:
- net GND: no longer J2.30
- net at J2.5: now also J1.5 (GP3); no longer J1.1 (GP0)
- net at J2.6: now also J1.4 (GP2); no longer J1.2 (GP1)
- net at J2.7: now also J1.2 (GP1); no longer J1.4 (GP2)
- net at J2.8: now also J1.1 (GP0); no longer J1.5 (GP3)
