File: pcb_picokeyboard.kicad_pcb (KiCad board)
At the start: 2 copper layers, 9 parts, among them J1 PICO, J2 502790-3091

Commit message: 2
Parts:
- J2: moved to B.Cu
- moved TP3 29.5 mm to (133.1, 86.8), turned to 90 degrees
- moved J2 25.1 mm to (116.9, 96.3)
- moved TP2 24.5 mm to (133.1, 83.3), turned to 90 degrees
- moved TP5 19.6 mm to (133.1, 79.7), turned to 90 degrees
- moved TP4 14.7 mm to (133.1, 76.2), turned to 90 degrees
- moved TP7 9.92 mm to (133.1, 72.6), turned to 90 degrees
- moved TP6 5.58 mm to (133.1, 69.1), turned to 90 degrees
- moved TP1 3.79 mm to (133.1, 65.5), turned to 90 degrees
Connections:
- J2 pad 30: GND -> unconnected-(J2-Pad30)
- J2 pad 5: Net-(J1-Pad1) -> Net-(J1-Pad5)
- J2 pad 6: Net-(J1-Pad2) -> Net-(J1-Pad4)
- J2 pad 7: Net-(J1-Pad4) -> Net-(J1-Pad2)
- J2 pad 8: Net-(J1-Pad5) -> Net-(J1-Pad1)
Routing:
- net Net-(J1-Pad1): track 0.00 -> 37.0 mm, vias 0 -> 1
- net Net-(J1-Pad2): track 0.00 -> 33.1 mm, vias 0 -> 1
- net Net-(J1-Pad4): track 0.00 -> 26.8 mm, vias 0 -> 1
- net Net-(J1-Pad5): track 0.00 -> 23.1 mm, vias 0 -> 1
- net Net-(J1-Pad6): track 0.00 -> 21.2 mm, vias 0 -> 1
- net Net-(J1-Pad20): track 0.00 -> 20.3 mm, vias 0 -> 1
- net Net-(J1-Pad7): track 0.00 -> 19.4 mm, vias 0 -> 1
- net Net-(J1-Pad19): track 0.00 -> 18.6 mm, vias 0 -> 1
- net Net-(J1-Pad9): track 0.00 -> 15.1 mm, vias 0 -> 1
- net Net-(J1-Pad17): track 0.00 -> 14.2 mm, vias 0 -> 1
- net Net-(J1-Pad10): track 0.00 -> 13.5 mm, vias 0 -> 1
- net Net-(J1-Pad16): track 0.00 -> 12.4 mm, vias 0 -> 1
- net Net-(J1-Pad11): track 0.00 -> 11.8 mm, vias 0 -> 1
- net Net-(J1-Pad15): track 0.00 -> 10.6 mm, vias 0 -> 1
- net Net-(J1-Pad12): track 0.00 -> 10.1 mm, vias 0 -> 1
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Other:
- board outline added: 26.3 x 49.9 mm
- copper layers 2 -> 8

Commit message: 3
Parts:
- moved TP2 19.5 mm to (120.5, 68.5)
- moved TP3 19.4 mm to (120.5, 72.0)
- moved TP4 12.6 mm to (120.5, 75.6)
- moved TP1 12.6 mm to (120.5, 65.2)
Routing:
- net Net-(J1-Pad32): track 0.00 -> 20.4 mm, vias 0 -> 1
- net Net-(J1-Pad31): track 0.00 -> 18.8 mm, vias 0 -> 1
- net Net-(J1-Pad21): track 0.00 -> 16.3 mm, vias 0 -> 1
- net Net-(J1-Pad22): track 0.00 -> 15.4 mm, vias 0 -> 1
- net Net-(J1-Pad29): track 0.00 -> 14.4 mm, vias 0 -> 1
- net Net-(J1-Pad24): track 0.00 -> 11.9 mm, vias 0 -> 1
- net Net-(J1-Pad27): track 0.00 -> 11.7 mm, vias 0 -> 1
- net Net-(J1-Pad25): track 0.00 -> 11.1 mm, vias 0 -> 1
- net Net-(J1-Pad26): track 0.00 -> 10.9 mm, vias 0 -> 1
- net Net-(J1-Pad1): track 37.0 -> 37.7 mm
- net GND: vias 0 -> 4
- added copper zone on B.Cu, net GND
- added copper zone on F.Cu, net GND
